File: module_5_1/relay_expander/relay_expander.kicad_sch (KiCad schematic)
At the start: 52 parts, among them J1 PLS-4, J2 2EDGR-5.08-05P, J3 2EDGR-5.08-04P, J4 2EDGR-5.08-02P, J5 2EDGR-5.08-02P, K1 HF49FD/024-1H12, K2 HF49FD/024-1H12, K3 HF49FD/024-1H12, K4 HF49FD/024-1H12, K5 HF49FD/024-1H12, K6 HF49FD/024-1H12, K7 HF49FD/024-1H12, Q1 AO3401A, U1 STM32G030F6Px, U2 ULN2003A, U3 MP1584, U4 AMS1117-3.3, U5 MAX3078E

Commit message: Gournd planes on DC-DC convertor have been fixed. Labels have been placed to be seen. An easter egg has been added.
Parts:
- C1, C5: LCSC Part (none) -> C14663; MPM CL10B104JA8NNNC -> (none); MPN (none) -> CL10B104JA8NNNC
- C2, C8: LCSC Part (none) -> C12891; MPM CL31X476KQHNNNE -> (none); MPN (none) -> CL31X476KQHNNNE
- C3, C7: LCSC Part (none) -> C13585; MPM CL31B106KBHNNNE -> (none); MPN (none) -> CL31B106KBHNNNE
- C4: LCSC Part (none) -> C14663; MPM C1608C0G2E151J080AA -> (none); MPN (none) -> C1608C0G2E151J080AA
- C6: LCSC Part (none) -> C19666; MPM CL10A475KP8NNNC -> (none); MPN (none) -> CL10A475KP8NNNC
- C9: LCSC Part (none) -> C3340; MPM CS1V221M-CRF10 -> (none); MPN (none) -> CS1V221M-CRF10
- D1: LCSC Part (none) -> C8678; MPM SS34 -> (none); MPN (none) -> SS34
- D2: LCSC Part (none) -> C283899; MPM SMAJ28A-TR -> (none); MPN (none) -> SMAJ28A-TR
- D3: LCSC Part (none) -> C118044; MPM BZX384-B10.115 -> (none); MPN (none) -> BZX384-B10.115
- D4: LCSC Part (none) -> C32677; MPM SM712 -> (none); MPN (none) -> SM712
- D5: MPM KT-SMD1206-G -> (none); MPN (none) -> KT-SMD1206-G
- F1: MPM FUSE 1A 250V 3X10 -> (none); MPN (none) -> FUSE 1A 250V 3X10; now not fitted
- FB1, FB2: LCSC Part (none) -> C1015; MPM BLM21AJ601SN1D -> (none); MPN (none) -> BLM21AJ601SN1D
- J1: MPM CL10B104JA8NNNC -> (none); MPN (none) -> CL10B104JA8NNNC; now not fitted
- J2: MPM 2EDGR-5.08-05P-14-00AH -> (none); MPN (none) -> 2EDGR-5.08-05P-14-00AH; now not fitted
- J3: MPM 2EDGR-5.08-04P-14-00AH -> (none); MPN (none) -> 2EDGR-5.08-04P-14-00AH; now not fitted
- J4, J5: MPM 2EDGR-5.08-02P-14-00AH -> (none); MPN (none) -> 2EDGR-5.08-02P-14-00AH; now not fitted
- JP2, JP3, JP4: now not fitted
- K1, K2, K3, K4, K5, K6, K7: MPM HF49FD/024-1H12 -> (none); MPN HF49FD/024-1H12 -> HF49FD/024-1H12; now not fitted
- L1: LCSC Part (none) -> C182159; MPM SMD0650_4u7H -> (none); MPN (none) -> SMD0650_4u7H
- Q1: LCSC Part (none) -> C15127; MPM AO3401A -> (none); MPN (none) -> AO3401A
- R1, R12, R5, R6: LCSC Part (none) -> C14675; MPM RC0603FR-07100KL -> (none); MPN (none) -> RC0603FR-07100KL
- R10, R13, R9: LCSC Part (none) -> C23204; MPM RC03K3561JT-KOME -> (none); MPN (none) -> RC03K3561JT-KOME
- R11: LCSC Part (none) -> C22787; MPM RC0603JR-07120RL -> (none); MPN (none) -> RC0603JR-07120RL
- R2: LCSC Part (none) -> C22952; MPM RC0805FR-210K-Hitano -> (none); MPN (none) -> RC0805FR-210K-Hitano
- R3: LCSC Part (none) -> C25962; MPM SMD 24.9K 0805 1% -> (none); MPN (none) -> SMD 24.9K 0805 1%
- R4: LCSC Part (none) -> C12447; MPM RC0603FR-40K2R-Hitano -> (none); MPN (none) -> RC0603FR-40K2R-Hitano
- R7: LCSC Part (none) -> C22975; MPM RC0603FR-072KL -> (none); MPN (none) -> RC0603FR-072KL
- R8: LCSC Part (none) -> C14676; MPM RC0603FR-071KL -> (none); MPN (none) -> RC0603FR-071KL
- U1: LCSC Part (none) -> C724040; MPM STM32G030F6P6TR -> (none); MPN (none) -> STM32G030F6P6TR
- U2: LCSC Part (none) -> C7512; MPM ULN2003ADR -> (none); MPN (none) -> ULN2003ADR
- U3: LCSC Part (none) -> C49367328; MPM MP1584EN -> (none); MPN (none) -> MP1584EN
- U4: LCSC Part (none) -> C6186; MPM AMS1117-3.3 -> (none); MPN (none) -> AMS1117-3.3
- U5: LCSC Part (none) -> C12545; MPM SP485REN-L/TR -> (none); MPN (none) -> SP485REN-L/TR
